Commit message: fixed jackal laser config in noetic

File: multi_jackal_description/urdf/base_accessories.urdf.xacro (robot description, xacro)
@@ -1,4 +1,4 @@
 <?xml version="1.0"?>
-<robot xmlns:xacro="http://www.ros.org/wiki/xacro">
+<robot xmlns:xacro="http://ros.org/wiki/xacro">
   <!-- Macros to generate standoffs for offset payload mounting. -->
   <xacro:include filename="accessories/standoffs.urdf.xacro" />
@@ -6,13 +6,81 @@
   <xacro:include filename="accessories/bridge_plate.urdf.xacro" />
   <!-- If enabled, generate the LASER payload (by default, a SICK LMS111). -->
-  <xacro:include filename="accessories/sick_lms1xx_mount.urdf.xacro" />
   <xacro:if value="$(optenv JACKAL_LASER 0)">
-    <sick_lms1xx_mount prefix="$(optenv JACKAL_LASER_MOUNT front)"
-                       topic="$(optenv JACKAL_LASER_TOPIC front/scan)"/>
-    <joint name="$(optenv JACKAL_LASER_MOUNT front)_laser_mount_joint" type="fixed">
-      <origin xyz="$(optenv JACKAL_LASER_OFFSET 0 0 0)"
-              rpy="$(optenv JACKAL_LASER_RPY 0 0 0)" />
-      <parent link="$(optenv JACKAL_LASER_MOUNT front)_mount" />
-      <child link="$(optenv JACKAL_LASER_MOUNT front)_laser_mount" />
+    <link name="front_laser">
+      <inertial>
+        <mass value="1.1" />
+        <origin xyz="0 0 0" />
+        <inertia ixx="${0.0833333 * 1.1 * (0.102*0.102 + 0.152*0.152)}" ixy="0.0" ixz="0.0"
+          iyy="${0.0833333 * 1.1 * (0.105*0.105 + 0.152*0.152)}" iyz="0.0"
+          izz="${0.0833333 * 1.1 * (0.105*0.105 + 0.102*0.102)}" />
+      </inertial>
+      <visual>
+        <origin xyz="0 0 0" rpy="0 0 0" />
+        <geometry>
+          <mesh filename="package://lms1xx/meshes/sick-lms1xx.dae" />
+        </geometry>
+      </visual>
+      <collision>
+        <origin xyz="0 0 -0.05" rpy="0 0 0" />
+        <geometry>
+          <box size="0.105 0.1 0.1" />
+        </geometry>
+      </collision>
+    </link>
+    <gazebo reference="front_laser">
+      <turnGravityOff>true</turnGravityOff>
+      <sensor type="ray" name="front_laser">
+        <pose>0 0 0 0 0 0</pose>
+        <visualize>false</visualize>
+        <update_rate>50</update_rate>
+        <ray>
+          <scan>
+            <horizontal>
+              <samples>720</samples>
+              <resolution>1</resolution>
+              <min_angle>-2.35619</min_angle>
+              <max_angle>2.35619</max_angle>
+            </horizontal>
+          </scan>
+          <range>
+            <min>0.1</min>
+            <max>30</max>
+            <resolution>0.01</resolution>
+          </range>
+          <noise>
+            <type>gaussian</type>
+            <mean>0.0</mean>
+            <stddev>0.001</stddev>
+          </noise>
+        </ray>
+        <plugin name="gazebo_ros_laser" filename="libgazebo_ros_laser.so">
+          <topicName>front/scan</topicName>
+          <frameName>front_laser</frameName>
+          <robotNamespace>jackal0</robotNamespace>
+        </plugin>
+      </sensor>
+    </gazebo>
+    <link name="front_laser_mount">
+      <visual>
+        <origin xyz="0 0 0" rpy="0 0 0" />
+        <geometry>
+          <mesh filename="package://multi_jackal_description/meshes/sick-lms1xx-bracket.stl" />
+        </geometry>
+        <material name="dark_grey" />
+      </visual>
+    </link>
+    <joint name="front_laser_joint" type="fixed">
+      <origin xyz="0 0 0.149" rpy="0 0 0" />
+      <parent link="front_laser_mount" />
+      <child link="front_laser" />
+    </joint>
+    <gazebo reference="front_laser_mount">
+      <material>Gazebo/DarkGrey</material>
+    </gazebo>
+    <joint name="front_laser_mount_joint" type="fixed">
+      <origin xyz="0 0 0"
+              rpy="0 0 0" />
+      <parent link="front_mount" />
+      <child link="front_laser_mount" />
     </joint>
   </xacro:if>
