Commit message: Remove unwanted parts from urdf file

File: multi_jackal_description/urdf/jackal.urdf.xacro (robot description, xacro)
@@ -3,21 +3,30 @@
      into Gazebo using robot state publisher.
      Requires the arguments: $namespace, $id -->
-<robot name="jackal" xmlns:xacro="http://ros.org/wiki/xacro">
-  <xacro:property name="PI"                        value="3.1415926535897931" />
-  <xacro:property name="wheelbase"                 value="0.262" />
-  <xacro:property name="track"                     value="0.37559" />
-  <xacro:property name="wheel_vertical_offset"     value="0.0345" />
+<robot name="jackal"
+  xmlns:xacro="http://ros.org/wiki/xacro">
+  <xacro:property name="PI" value="3.1415926535897931" />
+  <xacro:property name="wheelbase" value="0.262" />
+  <xacro:property name="track" value="0.37559" />
+  <xacro:property name="wheel_vertical_offset" value="0.0345" />
   <xacro:property name="footprint_vertical_offset" value="-0.0655" />
-  <xacro:property name="wheel_radius"              value="0.098" />
-  <xacro:property name="wheel_width"               value="0.040" />
-  <xacro:property name="chassis_length"            value="0.420" />
-  <xacro:property name="chassis_width"             value="0.310" />
-  <xacro:property name="chassis_height"            value="0.184" />
-  <xacro:property name="dummy_inertia"             value="1e-09"/>
-  <xacro:property name="mount_spacing"             value="0.120" />
-  <material name="dark_grey"><color rgba=" 0.2 0.2 0.2 1.0" /></material>
-  <material name="light_grey"><color rgba="0.4 0.4 0.4 1.0" /></material>
-  <material name="yellow"><color rgba="0.8 0.8 0.0 1.0" /></material>
-  <material name="black"><color rgba="0.15 0.15 0.15 1.0" /></material>
+  <xacro:property name="wheel_radius" value="0.098" />
+  <xacro:property name="wheel_width" value="0.040" />
+  <xacro:property name="chassis_length" value="0.420" />
+  <xacro:property name="chassis_width" value="0.310" />
+  <xacro:property name="chassis_height" value="0.184" />
+  <xacro:property name="dummy_inertia" value="1e-09"/>
+  <xacro:property name="mount_spacing" value="0.120" />
+  <material name="dark_grey">
+    <color rgba=" 0.2 0.2 0.2 1.0" />
+  </material>
+  <material name="light_grey">
+    <color rgba="0.4 0.4 0.4 1.0" />
+  </material>
+  <material name="yellow">
+    <color rgba="0.8 0.8 0.0 1.0" />
+  </material>
+  <material name="black">
+    <color rgba="0.15 0.15 0.15 1.0" />
+  </material>
   <!-- The wheel template. -->
   <xacro:macro name="wheel" params="prefix *joint_pose">
@@ -39,8 +48,5 @@
         <origin xyz="0 0 0" rpy="0 0 0"/>
         <mass value="0.477"/>
-        <inertia
-          ixx="0.0013" ixy="0" ixz="0"
-          iyy="0.0024" iyz="0"
-          izz="0.0013"/>
+        <inertia ixx="0.0013" ixy="0" ixz="0" iyy="0.0024" iyz="0" izz="0.0013"/>
       </inertial>
     </link>
@@ -104,11 +110,8 @@
       <mass value="16.523"/>
       <!-- Moments of inertia: ( chassis without wheels ) -->
-      <inertia
-        ixx="0.3136" ixy="-0.0008" ixz="0.0164"
-        iyy="0.3922" iyz="-0.0009"
-        izz="0.4485"/>
-      </inertial>
-  </link>
-  <link name="chefs_hat_link">
+      <inertia ixx="0.3136" ixy="-0.0008" ixz="0.0164" iyy="0.3922" iyz="-0.0009" izz="0.4485"/>
+    </inertial>
+  </link>
+  <!-- <link name="chefs_hat_link">
     <visual>
       <origin xyz="-0.34 0 0.25" rpy="0 ${-PI/2} ${PI}"/>
@@ -120,15 +123,13 @@
     <collision>
       <origin xyz="-0.34 0 0.25" rpy="0 ${-PI/2} ${PI}"/>
-      <!-- <origin xyz="-0.055 0 0.5"/> -->
       <geometry>
           <mesh filename="package://multi_jackal_description/meshes/ears_frame.stl"/>
-        <!-- <box size="0.36 0.34 0.4"/> -->
       </geometry>
     </collision>
-  </link>
-  <joint name="chefs_hat_joint" type="fixed">
+  </link> -->
+  <!-- <joint name="chefs_hat_joint" type="fixed">
     <parent link="chassis_link" />
     <child link="chefs_hat_link" />
-  </joint>
+  </joint> -->
   <link name="fenders_link">
     <visual>
@@ -199,14 +200,14 @@
   <xacro:include filename="custom_accessories.urdf.xacro" />
   <gazebo>
-  <plugin name="p3d_base_controller" filename="libgazebo_ros_p3d.so">
-    <alwaysOn>true</alwaysOn>
-    <updateRate>50.0</updateRate>
-    <bodyName>base_link</bodyName>
-    <topicName>base_pose_ground_truth</topicName>
-    <gaussianNoise>0.00</gaussianNoise>
-    <frameName>world</frameName>
-    <xyzOffsets>0 0 0</xyzOffsets>
-    <rpyOffsets>0 0 0</rpyOffsets>
-  </plugin>
-</gazebo>
+    <plugin name="p3d_base_controller" filename="libgazebo_ros_p3d.so">
+      <alwaysOn>true</alwaysOn>
+      <updateRate>50.0</updateRate>
+      <bodyName>base_link</bodyName>
+      <topicName>base_pose_ground_truth</topicName>
+      <gaussianNoise>0.00</gaussianNoise>
+      <frameName>world</frameName>
+      <xyzOffsets>0 0 0</xyzOffsets>
+      <rpyOffsets>0 0 0</rpyOffsets>
+    </plugin>
+  </gazebo>
 </robot>
