Commit message: fixed sick laser xacro include

File: multi_jackal_description/urdf/accessories/sick_lms1xx_mount.urdf.xacro (robot description, xacro)
@@ -28,5 +28,5 @@
   <xacro:include filename="$(find lms1xx)/urdf/sick_lms1xx.urdf.xacro" />
   <xacro:macro name="sick_lms1xx_mount" params="prefix topic">
-    <sick_lms1xx frame="${prefix}_laser" topic="${topic}" robot_namespace="$(arg namespace)" />
+    <xacro:sick_lms1xx frame="${prefix}_laser" topic="${topic}" robot_namespace="$(arg namespace)" />
     <link name="${prefix}_laser_mount">
       <visual>

File: multi_jackal_description/urdf/base_accessories.urdf.xacro (robot description, xacro)
@@ -6,81 +6,14 @@
   <xacro:include filename="accessories/bridge_plate.urdf.xacro" />
   <!-- If enabled, generate the LASER payload (by default, a SICK LMS111). -->
+  <xacro:include filename="accessories/sick_lms1xx_mount.urdf.xacro" />
   <xacro:if value="$(optenv JACKAL_LASER 0)">
-    <link name="front_laser">
-      <inertial>
-        <mass value="1.1" />
-        <origin xyz="0 0 0" />
-        <inertia ixx="${0.0833333 * 1.1 * (0.102*0.102 + 0.152*0.152)}" ixy="0.0" ixz="0.0"
-          iyy="${0.0833333 * 1.1 * (0.105*0.105 + 0.152*0.152)}" iyz="0.0"
-          izz="${0.0833333 * 1.1 * (0.105*0.105 + 0.102*0.102)}" />
-      </inertial>
-      <visual>
-        <origin xyz="0 0 0" rpy="0 0 0" />
-        <geometry>
-          <mesh filename="package://lms1xx/meshes/sick-lms1xx.dae" />
-        </geometry>
-      </visual>
-      <collision>
-        <origin xyz="0 0 -0.05" rpy="0 0 0" />
-        <geometry>
-          <box size="0.105 0.1 0.1" />
-        </geometry>
-      </collision>
-    </link>
-    <gazebo reference="front_laser">
-      <turnGravityOff>true</turnGravityOff>
-      <sensor type="ray" name="front_laser">
-        <pose>0 0 0 0 0 0</pose>
-        <visualize>false</visualize>
-        <update_rate>50</update_rate>
-        <ray>
-          <scan>
-            <horizontal>
-              <samples>720</samples>
-              <resolution>1</resolution>
-              <min_angle>-2.35619</min_angle>
-              <max_angle>2.35619</max_angle>
-            </horizontal>
-          </scan>
-          <range>
-            <min>0.1</min>
-            <max>30</max>
-            <resolution>0.01</resolution>
-          </range>
-          <noise>
-            <type>gaussian</type>
-            <mean>0.0</mean>
-            <stddev>0.001</stddev>
-          </noise>
-        </ray>
-        <plugin name="gazebo_ros_laser" filename="libgazebo_ros_laser.so">
-          <topicName>front/scan</topicName>
-          <frameName>front_laser</frameName>
-          <robotNamespace>jackal0</robotNamespace>
-        </plugin>
-      </sensor>
-    </gazebo>
-    <link name="front_laser_mount">
-      <visual>
-        <origin xyz="0 0 0" rpy="0 0 0" />
-        <geometry>
-          <mesh filename="package://multi_jackal_description/meshes/sick-lms1xx-bracket.stl" />
-        </geometry>
-        <material name="dark_grey" />
-      </visual>
-    </link>
-    <joint name="front_laser_joint" type="fixed">
-      <origin xyz="0 0 0.149" rpy="0 0 0" />
-      <parent link="front_laser_mount" />
-      <child link="front_laser" />
-    </joint>
-    <gazebo reference="front_laser_mount">
-      <material>Gazebo/DarkGrey</material>
-    </gazebo>
-    <joint name="front_laser_mount_joint" type="fixed">
-      <origin xyz="0 0 0"
-              rpy="0 0 0" />
-      <parent link="front_mount" />
-      <child link="front_laser_mount" />
+    <xacro:sick_lms1xx_mount prefix="$(optenv JACKAL_LASER_MOUNT front)"
+                       topic="$(optenv JACKAL_LASER_TOPIC front/scan)"/>
+    <!-- <link name="$(optenv JACKAL_LASER_MOUNT front)_laser_mount"></link> -->
+    <joint name="$(optenv JACKAL_LASER_MOUNT front)_laser_mount_joint" type="fixed">
+      <origin xyz="$(optenv JACKAL_LASER_OFFSET 0 0 0)"
+              rpy="$(optenv JACKAL_LASER_RPY 0 0 0)" />
+      <parent link="$(optenv JACKAL_LASER_MOUNT front)_mount" />
+      <child link="$(optenv JACKAL_LASER_MOUNT front)_laser_mount" />
     </joint>
   </xacro:if>

Commit message: Added frame and charging plug

File: multi_jackal_description/urdf/accessories/sick_lms1xx_mount.urdf.xacro (robot description, xacro)
@@ -27,6 +27,6 @@
 <robot xmlns:xacro="http://www.ros.org/wiki/xacro">
   <xacro:include filename="$(find lms1xx)/urdf/sick_lms1xx.urdf.xacro" />
-  <xacro:macro name="sick_lms1xx_mount" params="prefix topic">
-    <sick_lms1xx frame="${prefix}_laser" topic="${topic}" robot_namespace="$(arg namespace)" />
+  <xacro:macro name="sick_lms1xx_mount" params="prefix topic min_angle max_angle">
+    <sick_lms1xx frame="${prefix}_laser" topic="${topic}" robot_namespace="$(arg namespace)" min_angle="${min_angle}" max_angle="${max_angle}"/>
     <link name="${prefix}_laser_mount">
       <visual>

File: multi_jackal_description/urdf/base_accessories.urdf.xacro (robot description, xacro)
@@ -9,5 +9,7 @@
   <xacro:if value="$(optenv JACKAL_LASER 0)">
     <sick_lms1xx_mount prefix="$(optenv JACKAL_LASER_MOUNT front)"
-                       topic="$(optenv JACKAL_LASER_TOPIC front/scan)"/>
+                       topic="$(optenv JACKAL_LASER_TOPIC front/scan)"
+                       min_angle="-1.4"
+                       max_angle="1.4" />
     <joint name="$(optenv JACKAL_LASER_MOUNT front)_laser_mount_joint" type="fixed">
       <origin xyz="$(optenv JACKAL_LASER_OFFSET 0 0 0)"

File: multi_jackal_description/urdf/jackal.urdf.xacro (robot description, xacro)
@@ -110,4 +110,25 @@
       </inertial>
   </link>
+  <link name="chefs_hat_link">
+    <visual>
+      <origin xyz="-0.34 0 0.25" rpy="0 ${-PI/2} ${PI}"/>
+      <geometry>
+        <mesh filename="package://multi_jackal_description/meshes/ears_frame.stl"/>
+      </geometry>
+      <material name="black" />
+    </visual>
+    <collision>
+      <origin xyz="-0.34 0 0.25" rpy="0 ${-PI/2} ${PI}"/>
+      <!-- <origin xyz="-0.055 0 0.5"/> -->
+      <geometry>
+          <mesh filename="package://multi_jackal_description/meshes/ears_frame.stl"/>
+        <!-- <box size="0.36 0.34 0.4"/> -->
+      </geometry>
+    </collision>
+  </link>
+  <joint name="chefs_hat_joint" type="fixed">
+    <parent link="chassis_link" />
+    <child link="chefs_hat_link" />
+  </joint>
   <link name="fenders_link">
     <visual>
